File: PCB/Quaero.kicad_pcb (KiCad board)
At the start: 2 copper layers, 191.6 x 135.5 mm, 65 parts, among them J1 USB_C_Receptacle_USB2.0_16P, J2 OLED_128x32, U1 RP2040_Zero

Commit message: Safety commit before flipping rp2040
Parts:
- added H10: MountingHole_Pad, MountingHole:MountingHole_2.2mm_M2_Pad, F.Cu at (84.8, 86.1)
- added H7: MountingHole_Pad, MountingHole:MountingHole_2.2mm_M2_Pad, F.Cu at (108.9, 61.1)
- added H8: MountingHole_Pad, MountingHole:MountingHole_2.2mm_M2_Pad, F.Cu at (86.2, 138.3)
- added H9: MountingHole_Pad, MountingHole:MountingHole_2.2mm_M2_Pad, F.Cu at (154.0, 151.6)
- H1, H2, H3, H4, H5, H6: footprint MountingHole:MountingHole_2.2mm_M2_DIN965_Pad -> MountingHole:MountingHole_2.2mm_M2_Pad
- moved H5 172.6 mm to (40.7, 111.3)
- moved H1 166.1 mm to (38.9, 93.3)
- moved H2 158.6 mm to (43.4, 131.1)
- moved H4 110.7 mm to (107.7, 81.8)
- moved H3 100.7 mm to (106.7, 122.3)
- moved H6 65.9 mm to (150.9, 107.1)
- moved U1 6.48 mm to (160.9, 90.8)
- moved J2 5.46 mm to (153.6, 119.1)
- moved J1 5.25 mm to (162.8, 130.3)
- moved D7 0.35 mm to (39.5, 97.0)
Connections:
- J1 pad A6: unconnected-(J1-D+-PadA6) -> RX
- J1 pad A7: unconnected-(J1-D--PadA7) -> TX
- J1 pad A8: TX -> unconnected-(J1-SBU1-PadA8)
- J1 pad B6: unconnected-(J1-D+-PadB6) -> RX
- J1 pad B7: unconnected-(J1-D--PadB7) -> TX
- J1 pad B8: TX -> unconnected-(J1-SBU2-PadB8)
Routing:
- net +5V: track 0.00 -> 63.6 mm
- net LRow-5: track 71.3 -> 117.0 mm
- net +3.3V: track 0.00 -> 42.8 mm
- net TX: track 0.00 -> 29.7 mm
- net RX: track 0.00 -> 28.3 mm
- net LRow-1: track 163.7 -> 137.3 mm
- net Net-(D13-A): track 0.00 -> 5.58 mm
- net LRow-4: track 135.1 -> 140.2 mm
- net LCol-1: track 199.6 -> 195.0 mm
- net LCol-2: track 179.4 -> 175.8 mm
- net LRow-2: track 149.7 -> 146.7 mm
- net LCol-6: track 120.5 -> 123.5 mm
- net LCol-5: track 135.9 -> 137.9 mm
- net LCol-3: track 187.2 -> 185.6 mm
- net SCL: track 15.8 -> 16.9 mm
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Other:
- board size 191.6 x 135.5 mm -> 159.7 x 127.4 mm

Commit message: Finished right side
Parts:
- added D29: Diode, Diode_THT:D_DO-35_SOD27_P7.62mm_Horizontal, B.Cu at (249.7, 65.1)
- added D30: Diode, Diode_THT:D_DO-35_SOD27_P7.62mm_Horizontal, B.Cu at (268.4, 62.2)
- added D31: Diode, Diode_THT:D_DO-35_SOD27_P7.62mm_Horizontal, B.Cu at (293.7, 53.6)
- added D32: Diode, Diode_THT:D_DO-35_SOD27_P7.62mm_Horizontal, B.Cu at (319.1, 63.0)
- added D33: Diode, Diode_THT:D_DO-35_SOD27_P7.62mm_Horizontal, B.Cu at (342.5, 77.8)
- added D34: Diode, Diode_THT:D_DO-35_SOD27_P7.62mm_Horizontal, B.Cu at (361.6, 80.3)
- added D35: Diode, Diode_THT:D_DO-35_SOD27_P7.62mm_Horizontal, B.Cu at (250.4, 84.2)
- added D36: Diode, Diode_THT:D_DO-35_SOD27_P7.62mm_Horizontal, B.Cu at (269.5, 81.2)
- added D37: Diode, Diode_THT:D_DO-35_SOD27_P7.62mm_Horizontal, B.Cu at (293.7, 72.6)
- added D38: Diode, Diode_THT:D_DO-35_SOD27_P7.62mm_Horizontal, B.Cu at (318.0, 82.0)
- added D39: Diode, Diode_THT:D_DO-35_SOD27_P7.62mm_Horizontal, B.Cu at (340.4, 96.6)
- added D40: Diode, Diode_THT:D_DO-35_SOD27_P7.62mm_Horizontal, B.Cu at (359.3, 99.6)
- added D41: Diode, Diode_THT:D_DO-35_SOD27_P7.62mm_Horizontal, B.Cu at (251.4, 104.2)
- added D42: Diode, Diode_THT:D_DO-35_SOD27_P7.62mm_Horizontal, B.Cu at (270.4, 100.9)
- added D43: Diode, Diode_THT:D_DO-35_SOD27_P7.62mm_Horizontal, B.Cu at (293.8, 92.9)
- added D44: Diode, Diode_THT:D_DO-35_SOD27_P7.62mm_Horizontal, B.Cu at (316.3, 102.3)
- added D45: Diode, Diode_THT:D_DO-35_SOD27_P7.62mm_Horizontal, B.Cu at (337.8, 116.9)
- added D46: Diode, Diode_THT:D_DO-35_SOD27_P7.62mm_Horizontal, B.Cu at (356.7, 119.3)
- added D47: Diode, Diode_THT:D_DO-35_SOD27_P7.62mm_Horizontal, B.Cu at (252.7, 122.2)
- added D48: Diode, Diode_THT:D_DO-35_SOD27_P7.62mm_Horizontal, B.Cu at (271.2, 119.5)
- added D49: Diode, Diode_THT:D_DO-35_SOD27_P7.62mm_Horizontal, B.Cu at (293.9, 110.8)
- added D50: Diode, Diode_THT:D_DO-35_SOD27_P7.62mm_Horizontal, B.Cu at (315.1, 120.7)
- added D51: Diode, Diode_THT:D_DO-35_SOD27_P7.62mm_Horizontal, B.Cu at (335.7, 134.6)
- added D52: Diode, Diode_THT:D_DO-35_SOD27_P7.62mm_Horizontal, B.Cu at (354.6, 137.5)
- added D53: Diode, Diode_THT:D_DO-35_SOD27_P7.62mm_Horizontal, B.Cu at (226.6, 161.7)
- added D54: Diode, Diode_THT:D_DO-35_SOD27_P7.62mm_Horizontal, B.Cu at (248.0, 148.1)
- added D55: Diode, Diode_THT:D_DO-35_SOD27_P7.62mm_Horizontal, B.Cu at (271.2, 142.3)
- added D56: Diode, Diode_THT:D_DO-35_SOD27_P7.62mm_Horizontal, B.Cu at (293.2, 142.6)
- added H1: MountingHole_Pad, MountingHole:MountingHole_2.2mm_M2_Pad, B.Cu at (359.6, 95.9)
- added H10: MountingHole_Pad, MountingHole:MountingHole_2.2mm_M2_Pad, B.Cu at (313.7, 88.7)
- added H2: MountingHole_Pad, MountingHole:MountingHole_2.2mm_M2_Pad, B.Cu at (355.1, 133.7)
- added H3: MountingHole_Pad, MountingHole:MountingHole_2.2mm_M2_Pad, B.Cu at (291.8, 124.9)
- added H4: MountingHole_Pad, MountingHole:MountingHole_2.2mm_M2_Pad, B.Cu at (290.8, 84.4)
- added H5: MountingHole_Pad, MountingHole:MountingHole_2.2mm_M2_Pad, B.Cu at (357.8, 113.9)
- added H6: MountingHole_Pad, MountingHole:MountingHole_2.2mm_M2_Pad, B.Cu at (247.6, 109.7)
- added H7: MountingHole_Pad, MountingHole:MountingHole_2.2mm_M2_Pad, B.Cu at (289.6, 63.7)
- added H8: MountingHole_Pad, MountingHole:MountingHole_2.2mm_M2_Pad, B.Cu at (312.3, 140.9)
- added H9: MountingHole_Pad, MountingHole:MountingHole_2.2mm_M2_Pad, B.Cu at (244.5, 154.2)
- added R-MCU1: RP2040_Zero, ScottoKeebs_MCU:RP2040_Zero_Flipped, F.Cu at (237.6, 93.4)
- added R-OLED1: OLED_128x32, ScottoKeebs_Components:OLED_128x32, F.Cu at (232.9, 122.3)
- added R-USB1: USB_C_Receptacle_USB2.0_16P, Connector_USB:USB_C_Receptacle_GCT_USB4085, F.Cu at (235.8, 133.4)
- added S29: Keyswitch, ai03_ks33hotswap:Gateron-KS33-Hotswap-1U, B.Cu at (259.4, 70.8)
- added S30: Keyswitch, ai03_ks33hotswap:Gateron-KS33-Hotswap-1U, B.Cu at (278.2, 67.3)
- added S31: Keyswitch, ai03_ks33hotswap:Gateron-KS33-Hotswap-1U, B.Cu at (303.2, 59.8)
- added S32: Keyswitch, ai03_ks33hotswap:Gateron-KS33-Hotswap-1U, B.Cu at (328.4, 69.7)
- added S33: Keyswitch, ai03_ks33hotswap:Gateron-KS33-Hotswap-1U, B.Cu at (351.4, 85.2)
- added S34: Keyswitch, ai03_ks33hotswap:Gateron-KS33-Hotswap-1U, B.Cu at (370.3, 87.5)
- added S35: Keyswitch, ai03_ks33hotswap:Gateron-KS33-Hotswap-1U, B.Cu at (260.4, 89.8)
- added S36: Keyswitch, ai03_ks33hotswap:Gateron-KS33-Hotswap-1U, B.Cu at (279.2, 86.3)
- added S37: Keyswitch, ai03_ks33hotswap:Gateron-KS33-Hotswap-1U, B.Cu at (303.2, 78.8)
- added S38: Keyswitch, ai03_ks33hotswap:Gateron-KS33-Hotswap-1U, B.Cu at (327.0, 88.7)
- added S39: Keyswitch, ai03_ks33hotswap:Gateron-KS33-Hotswap-1U, B.Cu at (349.0, 104.1)
- added S40: Keyswitch, ai03_ks33hotswap:Gateron-KS33-Hotswap-1U, B.Cu at (367.9, 106.4)
- added S41: Keyswitch, ai03_ks33hotswap:Gateron-KS33-Hotswap-1U, B.Cu at (261.3, 108.8)
- added S42: Keyswitch, ai03_ks33hotswap:Gateron-KS33-Hotswap-1U, B.Cu at (280.2, 105.3)
- added S43: Keyswitch, ai03_ks33hotswap:Gateron-KS33-Hotswap-1U, B.Cu at (303.2, 97.8)
- added S44: Keyswitch, ai03_ks33hotswap:Gateron-KS33-Hotswap-1U, B.Cu at (325.7, 107.8)
- added S45: Keyswitch, ai03_ks33hotswap:Gateron-KS33-Hotswap-1U, B.Cu at (346.7, 123.0)
- added S46: Keyswitch, ai03_ks33hotswap:Gateron-KS33-Hotswap-1U, B.Cu at (365.6, 125.3)
- added S47: Keyswitch, ai03_ks33hotswap:Gateron-KS33-Hotswap-1U, B.Cu at (262.3, 127.8)
- added S48: Keyswitch, ai03_ks33hotswap:Gateron-KS33-Hotswap-1U, B.Cu at (281.2, 124.3)
- added S49: Keyswitch, ai03_ks33hotswap:Gateron-KS33-Hotswap-1U, B.Cu at (303.2, 116.9)
- added S50: Keyswitch, ai03_ks33hotswap:Gateron-KS33-Hotswap-1U, B.Cu at (324.4, 126.8)
- added S51: Keyswitch, ai03_ks33hotswap:Gateron-KS33-Hotswap-1U, B.Cu at (344.4, 141.9)
- added S52: Keyswitch, ai03_ks33hotswap:Gateron-KS33-Hotswap-1U, B.Cu at (363.3, 144.2)
- added S53: Keyswitch, ai03_ks33hotswap:Gateron-KS33-Hotswap-1U, B.Cu at (237.8, 161.2)
- added S54: Keyswitch, ai03_ks33hotswap:Gateron-KS33-Hotswap-1U, B.Cu at (258.8, 151.4)
- added S55: Keyswitch, ai03_ks33hotswap:Gateron-KS33-Hotswap-1U, B.Cu at (280.7, 148.4)
- added S56: Keyswitch, ai03_ks33hotswap:Gateron-KS33-Hotswap-1U, B.Cu at (302.0, 149.6)
- L-MCU1: renamed from U1; footprint ScottoKeebs_MCU:RP2040_Zero -> ScottoKeebs_MCU:RP2040_Zero_Flipped
- moved L-USB1 6.44 mm to (162.4, 136.7)
- renumbered J2 to L-OLED1, J1 to L-USB1
Connections:
- net +3.3V renamed L +3.3V
- net +5V renamed L +5V
- net SCL renamed L-SCL
- net SDA renamed L-SDA
- L-MCU1 pad 10: RX -> LRow-4
- L-MCU1 pad 13: LRow-5 -> L-TX
- L-MCU1 pad 14: LRow-4 -> L-RX
- L-MCU1 pad 15: LCol-1 -> unconnected-(L-MCU1-14-Pad15)
- L-MCU1 pad 16: LCol-2 -> LRow-5
- L-MCU1 pad 17: LCol-3 -> unconnected-(L-MCU1-26-Pad17)
- L-MCU1 pad 18: LCol-4 -> unconnected-(L-MCU1-27-Pad18)
- L-MCU1 pad 19: LCol-5 -> unconnected-(L-MCU1-28-Pad19)
- L-MCU1 pad 20: LCol-6 -> unconnected-(L-MCU1-29-Pad20)
- L-MCU1 pad 4: unconnected-(U1-3-Pad4) -> LCol-6
- L-MCU1 pad 5: unconnected-(U1-4-Pad5) -> LCol-5
- L-MCU1 pad 6: unconnected-(U1-5-Pad6) -> LCol-4
- L-MCU1 pad 7: unconnected-(U1-6-Pad7) -> LCol-3
- L-MCU1 pad 8: unconnected-(U1-7-Pad8) -> LCol-2
- L-MCU1 pad 9: TX -> LCol-1
- L-USB1 pad A6: RX -> L-RX
- L-USB1 pad A7: TX -> L-TX
- L-USB1 pad B6: RX -> L-RX
- L-USB1 pad B7: TX -> L-TX
Routing:
- net RCol-1: track 0.00 -> 197.3 mm, vias 0 -> 1
- net RCol-3: track 0.00 -> 186.7 mm, vias 0 -> 1
- net RCol-2: track 0.00 -> 178.9 mm, vias 0 -> 1
- net RCol-4: track 0.00 -> 168.0 mm, vias 0 -> 1
- net RRow-1: track 0.00 -> 163.4 mm
- net RRow-2: track 0.00 -> 143.3 mm
- net RRow-4: track 0.00 -> 136.9 mm
- net RCol-5: track 0.00 -> 135.8 mm, vias 0 -> 1
- net RRow-3: track 0.00 -> 130.7 mm
- net RCol-6: track 0.00 -> 120.1 mm, vias 0 -> 1
- net RRow-5: track 0.00 -> 118.0 mm
- net R +5V: track 0.00 -> 65.0 mm
- net R-RX: track 0.00 -> 39.3 mm
- net GND: track 0.00 -> 37.7 mm, vias 0 -> 55
- net R-TX: track 0.00 -> 36.9 mm
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- added copper zone on B.Cu, net GND
- added copper zone on F.Cu, net GND
Other:
- board size 159.7 x 127.4 mm -> 366.1 x 130 mm

Commit message: Final PCB
Parts:
- added mouse-bite-5mm-slot: VAL**, marbastlib-various:mouse-bite-5mm-slot, F.Cu at (199.7, 127.8)
- added mouse-bite-5mm-slot: VAL**, marbastlib-various:mouse-bite-5mm-slot, F.Cu at (199.7, 62.6)
- moved D4 188.7 mm to (293.3, 42.5), turned to -97 degrees
- moved S4 188.1 mm to (283.1, 47.4), turned to 173 degrees
- moved D31 187.9 mm to (106.1, 42.6), turned to -83 degrees
- moved D3 187.9 mm to (266.5, 48.8), turned to -93 degrees
- moved H7 187.4 mm to (296.2, 53.0), turned to -7 degrees
- moved D5 187.4 mm to (317.1, 53.7), turned to -100 degrees
- moved S31 187.3 mm to (116.3, 47.5), turned to -173 degrees
- moved S3 187.2 mm to (256.9, 54.3), turned to 177 degrees
- moved D32 187.2 mm to (132.4, 48.8), turned to -87 degrees
- moved S5 186.9 mm to (307.0, 57.9), turned to 170 degrees
- moved D6 186.8 mm to (335.8, 59.3), turned to -100 degrees
- moved H7 186.7 mm to (103.2, 53.1), turned to -173 degrees
- moved D30 186.6 mm to (82.0, 54.2), turned to -80 degrees
- moved S32 186.5 mm to (142.4, 54.4), turned to -177 degrees
- moved D1 186.5 mm to (222.8, 60.8), turned to -90 degrees
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Other:
- board size 366.1 x 130 mm -> 312.5 x 136 mm

Commit message: added files + readme improvements
Parts:
- moved D26 36.2 mm to (311.6, 168.9)
- moved H9 36.2 mm to (76.3, 184.0)
- moved D25 36.2 mm to (289.8, 166.5)
- moved H9 36.2 mm to (336.6, 183.9)
- moved S53 36.2 mm to (70.5, 191.8)
- moved D15 36.2 mm to (271.4, 122.3)
- moved D23 36.2 mm to (313.7, 148.1)
- moved D33 36.2 mm to (164.2, 96.3)
- moved D36 36.2 mm to (92.2, 108.5)
- moved D37 36.2 mm to (115.2, 97.0)
- moved D39 36.2 mm to (164.5, 115.1)
- moved D48 36.2 mm to (98.6, 146.3)
- moved D50 36.2 mm to (142.3, 142.2)
- moved D8 36.2 mm to (248.6, 115.3)
- moved H1 36.2 mm to (183.4, 112.1)
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